Commit message: make working version

File: ros_solid/urdf/ros_solid copy 2.urdf (robot description, URDF)
Before this commit: robot rozum_pulse_75, 14 links, 14 joints
Links:
- removed link link1_dummy
- removed link link2_dummy
- removed link link3_dummy
- removed link link4_dummy
- removed link link5_dummy
- removed link link6_dummy
- removed link world
Joints:
- removed joint gripper_joint
- removed joint joint1_post_transform
- removed joint joint2_post_transform
- removed joint joint3_post_transform
- removed joint joint4_post_transform
- removed joint joint5_post_transform
- removed joint joint6_post_transform
- removed joint world_joint
- joint joint1: child link1_dummy -> link1; origin xyz=0.0 0.0 0.0 rpy=0 0 0 -> xyz=0.0 0.0 0.215 rpy=1.5707963 0 0
- joint joint2: child link2_dummy -> link2; origin xyz=0.0 0.0 0.0 rpy=0 0 0 -> xyz=-0.286 -0.0 0.119 rpy=0 0 0
- joint joint3: child link3_dummy -> link3; origin xyz=0.0 0.0 0.0 rpy=0 0 0 -> xyz=-0.26 -0.0 -0.093 rpy=0 0 0
- joint joint4: child link4_dummy -> link4; origin xyz=0.0 0.0 0.0 rpy=0 0 0 -> xyz=0.0 0.0 0.093 rpy=1.5707963 0 0
- joint joint5: child link5_dummy -> link5; origin xyz=0.0 0.0 0.0 rpy=0 0 0 -> xyz=0.0 0.0 0.1681 rpy=-1.5707963 0 0
- joint joint6: child link6_dummy -> link6; origin xyz=0.0 0.0 0.0 rpy=0 0 0 -> xyz=0.0 0.0 0.1196 rpy=0 0 0

File: ros_solid/urdf/ros_solid copy 3.urdf (robot description, URDF)
Before this commit: robot rozum_pulse_75, 14 links, 14 joints
Links:
- removed link link1_dummy
- removed link link2_dummy
- removed link link3_dummy
- removed link link4_dummy
- removed link link5_dummy
- removed link link6_dummy
- removed link world
- added link tool_frame
Joints:
- removed joint gripper_joint
- removed joint joint1_post_transform
- removed joint joint2_post_transform
- removed joint joint3_post_transform
- removed joint joint4_post_transform
- removed joint joint5_post_transform
- removed joint joint6_post_transform
- removed joint world_joint
- added joint joint7: type fixed, parent link6, child tool_frame, origin xyz=0.0 0.0 0.1196 rpy=0 0 0
- joint joint1: child link1_dummy -> link1
- joint joint2: child link2_dummy -> link2; origin xyz=0.0 0.0 0.0 rpy=0 0 0 -> xyz=0.0 0.0 0.215 rpy=1.5707963 0 0
- joint joint3: child link3_dummy -> link3; origin xyz=0.0 0.0 0.0 rpy=0 0 0 -> xyz=-0.286 -0.0 0.119 rpy=0 0 0
- joint joint4: child link4_dummy -> link4; origin xyz=0.0 0.0 0.0 rpy=0 0 0 -> xyz=-0.26 -0.0 -0.093 rpy=0 0 0
- joint joint5: child link5_dummy -> link5; origin xyz=0.0 0.0 0.0 rpy=0 0 0 -> xyz=0.0 0.0 0.093 rpy=1.5707963 0 0
- joint joint6: child link6_dummy -> link6; origin xyz=0.0 0.0 0.0 rpy=0 0 0 -> xyz=0.0 0.0 0.1681 rpy=-1.5707963 0 0
