Commit message: fixed not loading error and robot crash

File: rozum_pulse_75_control/urdf/rozum_pulse_75_controllers.xacro (robot description, xacro)
@@ -1,5 +1,5 @@
 <?xml version="1.0" encoding="utf-8"?>
 <robot xmlns:xacro="http://www.ros.org/wiki/xacro">
-    <xacro:macro name="rozum75_ros2_control" params="name prefix use_mock_hardware:=false mock_sensor_commands:=false">
+    <xacro:macro name="rozum75_ros2_control" params="name prefix use_mock_hardware:=false mock_sensor_commands:=false base_url:=http://10.10.10.20:8081">
         <ros2_control name="${name}" type="system">
             <hardware>
@@ -13,5 +13,5 @@
                     <!-- Real hardware -->
                     <plugin>rozum_pulse_75_hardware/RozumSystemHardware</plugin>
-                    <param name="base_url">10.10.10.20</param>
+                    <param name="base_url">${base_url}</param>
                     <param name="command_interface">position</param>
                     <param name="joints_order">joint1,joint2,joint3,joint4,joint5,joint6</param>
@@ -22,10 +22,10 @@
             </hardware>
             <!-- Joint interfaces -->
-            <joint name="joint1"><command_interface name="position"/><state_interface name="position"/><state_interface name="velocity"/></joint>
-            <joint name="joint2"><command_interface name="position"/><state_interface name="position"/><state_interface name="velocity"/></joint>
-            <joint name="joint3"><command_interface name="position"/><state_interface name="position"/><state_interface name="velocity"/></joint>
-            <joint name="joint4"><command_interface name="position"/><state_interface name="position"/><state_interface name="velocity"/></joint>
-            <joint name="joint5"><command_interface name="position"/><state_interface name="position"/><state_interface name="velocity"/></joint>
-            <joint name="joint6"><command_interface name="position"/><state_interface name="position"/><state_interface name="velocity"/></joint>
+            <joint name="joint1"><command_interface name="position"/><state_interface name="position"/></joint>
+            <joint name="joint2"><command_interface name="position"/><state_interface name="position"/></joint>
+            <joint name="joint3"><command_interface name="position"/><state_interface name="position"/></joint>
+            <joint name="joint4"><command_interface name="position"/><state_interface name="position"/></joint>
+            <joint name="joint5"><command_interface name="position"/><state_interface name="position"/></joint>
+            <joint name="joint6"><command_interface name="position"/><state_interface name="position"/></joint>
         </ros2_control>
     </xacro:macro>
