Commit message: fixed gripper + delete old moveit conf

File: rozum_pulse_75_control/urdf/rozum_pulse_75_with_gripper.xacro (robot description, xacro)
@@ -7,6 +7,6 @@
     <xacro:arg name="mock_sensor_commands" default="false"/>
     <!-- import main macro -->
-    <!-- <xacro:include filename="$(find dh_ag95_description)/urdf/dh_ag95_macro.xacro" />
-    <xacro:include filename="$(find dh_gripper_driver)/urdf/dh_ag95.ros2_control.xacro" /> -->
+    <xacro:include filename="$(find dh_ag95_description)/urdf/dh_ag95_macro.xacro" />
+    <xacro:include filename="$(find dh_gripper_driver)/urdf/dh_ag95.ros2_control.xacro" />
     <xacro:include filename="$(find rozum_pulse_75)/urdf/rozum_pulse_75.xacro" />
     <xacro:include filename="$(find rozum_pulse_75_control)/urdf/rozum_pulse_75_controllers.xacro" />
@@ -19,3 +19,17 @@
     />
     <link name="gripper_base"/>
+    <!-- gripper -->
+    <xacro:dh_ag95_gripper
+        prefix=""
+        parent="gripper_base">
+        <origin xyz="0 0 0" rpy="0 0 -1.57079632679" />
+    </xacro:dh_ag95_gripper>
+    <!-- gripper ros2_control -->
+    <xacro:dh_ag95_gripper_ros2_control
+        name="dh_ag95_gripper"
+        prefix="$(arg prefix)"
+        com_port="$(arg com_port)"
+        use_mock_hardware="$(arg use_mock_hardware)"
+        mock_sensor_commands="$(arg mock_sensor_commands)"
+    />
 </robot>
