Commit message: fix moveit

File: new_moveit/config/rozum75_with_gripper.urdf.xacro (robot description, xacro)
@@ -4,6 +4,6 @@
     <!-- Import rozum75_with_gripper urdf file -->
     <xacro:include filename="$(find rozum_pulse_75_control)/urdf/rozum_pulse_75_with_gripper.xacro" />
-    <!-- Import control_xacro -->
+    <!-- Import control_xacro
     <xacro:include filename="rozum75_with_gripper.ros2_control.xacro" />
-    <xacro:rozum75_with_gripper_ros2_control name="FakeSystem" initial_positions_file="$(arg initial_positions_file)"/>
+    <xacro:rozum75_with_gripper_ros2_control name="FakeSystem" initial_positions_file="$(arg initial_positions_file)"/> -->
 </robot>

File: rozum_pulse_75/urdf/rozum_pulse_75.xacro (robot description, xacro)
@@ -149,7 +149,13 @@
     <axis
       xyz="0 0 1" />
-    <limit
+        <!-- <limit
       lower="-0.6108652382"
       upper="3.76991118431"
+      effort="10"
+      velocity="10" /> -->
+      <!-- commented out limits from DH file because they are too tight -->
+    <limit
+      lower="-3.14159265359"
+      upper="3.14159265359"
       effort="10"
       velocity="10" />
@@ -209,7 +215,12 @@
     <axis
       xyz="0 0 1" />
-    <limit
+    <!-- <limit
       lower="-0.6108652382"
       upper="3.76991118431"
+      effort="10"
+      velocity="10" /> -->
+    <limit
+      lower="-3.14159265359"
+      upper="3.14159265359"
       effort="10"
       velocity="10" />
