Commit message: add hardware interface: read

File: rozum_pulse_75/urdf/rozum_pulse_75.xacro (robot description, xacro)
@@ -5,4 +5,5 @@
 <robot
   name="rozum_pulse_75" xmlns:xacro="http://ros.org/wiki/xacro">
+  <xacro:arg name="rozum_base_url" default="http://10.10.10.20:8081"/>
   <xacro:include filename="$(find rozum_pulse_75)/urdf/ag95.xacro" />
   <link
@@ -528,3 +529,20 @@
       link="gripper_base" />
   </joint>
+  <ros2_control name="RozumSystem" type="system">
+    <hardware>
+      <plugin>rozum_pulse_75_hardware/RozumSystemHardware</plugin>
+      <param name="base_url">10.10.10.20</param>
+      <param name="command_interface">position</param>
+      <param name="joints_order">joint1,joint2,joint3,joint4,joint5,joint6</param>
+      <param name="write_speed_percent">20</param>
+      <param name="write_motion_type">JOINT</param>
+      <param name="use_pose_endpoint">true</param>
+    </hardware>
+    <joint name="joint1"><command_interface name="position"/><state_interface name="position"/><state_interface name="velocity"/></joint>
+    <joint name="joint2"><command_interface name="position"/><state_interface name="position"/><state_interface name="velocity"/></joint>
+    <joint name="joint3"><command_interface name="position"/><state_interface name="position"/><state_interface name="velocity"/></joint>
+    <joint name="joint4"><command_interface name="position"/><state_interface name="position"/><state_interface name="velocity"/></joint>
+    <joint name="joint5"><command_interface name="position"/><state_interface name="position"/><state_interface name="velocity"/></joint>
+    <joint name="joint6"><command_interface name="position"/><state_interface name="position"/><state_interface name="velocity"/></joint>
+  </ros2_control>
 </robot>

Commit message: demo initial

File: rozum_pulse_75/urdf/rozum_pulse_75.xacro (robot description, xacro)
@@ -47,5 +47,5 @@
   <link name="world" />
   <joint name="world_joint" type="fixed">
-    <origin xyz="0 0 0" rpy="0 0 0" />
+    <origin xyz="0 0 0" rpy="0 0 3.14159265359" />
     <parent link="world" />
     <child link="base_link" />

File: rozum_pulse_75_control/urdf/rozum_pulse_75_with_gripper.xacro (robot description, xacro)
@@ -7,6 +7,6 @@
     <xacro:arg name="mock_sensor_commands" default="false"/>
     <!-- import main macro -->
-    <xacro:include filename="$(find dh_ag95_description)/urdf/dh_ag95_macro.xacro" />
-    <xacro:include filename="$(find dh_gripper_driver)/urdf/dh_ag95.ros2_control.xacro" />
+    <!-- <xacro:include filename="$(find dh_ag95_description)/urdf/dh_ag95_macro.xacro" />
+    <xacro:include filename="$(find dh_gripper_driver)/urdf/dh_ag95.ros2_control.xacro" /> -->
     <xacro:include filename="$(find rozum_pulse_75)/urdf/rozum_pulse_75.xacro" />
     <xacro:include filename="$(find rozum_pulse_75_control)/urdf/rozum_pulse_75_controllers.xacro" />
@@ -19,17 +19,3 @@
     />
     <link name="gripper_base"/>
-    <!-- gripper -->
-    <xacro:dh_ag95_gripper
-        prefix=""
-        parent="gripper_base">
-        <origin xyz="0 0 0" rpy="0 0 -1.57079632679" />
-    </xacro:dh_ag95_gripper>
-    <!-- gripper ros2_control -->
-    <xacro:dh_ag95_gripper_ros2_control
-        name="dh_ag95_gripper"
-        prefix="$(arg prefix)"
-        com_port="$(arg com_port)"
-        use_mock_hardware="$(arg use_mock_hardware)"
-        mock_sensor_commands="$(arg mock_sensor_commands)"
-    />
 </robot>
